Commit message: Update robot core xacro and gamefield thin sdf.The robot's wheel separation and the gamefield are adjusted

File: src/ppp_bot/description/robot_core.xacro (robot description, xacro)
@@ -24,5 +24,5 @@
             <origin xyz="0.15 0 0.075"/>
             <geometry>
-                <box size="0.3 0.3 0.15"/>
+                <box size="0.3 0.24 0.15"/>
             </geometry>
             <material name="white"/>
@@ -31,8 +31,8 @@
             <origin xyz="0.15 0 0.075"/>
             <geometry>
-                <box size="0.3 0.3 0.15"/>
+                <box size="0.3 0.24 0.15"/>
             </geometry>
         </collision>
-        <xacro:inertial_box mass="0.5" x="0.3" y="0.3" z="0.15">
+        <xacro:inertial_box mass="0.5" x="0.3" y="0.24" z="0.15">
             <origin xyz="0.15 0 0.075" rpy="0 0 0"/>
         </xacro:inertial_box>
@@ -42,5 +42,5 @@
         <parent link="base_link"/>
         <child link="left_wheel"/>
-        <origin xyz="0 0.175 0" rpy="-${pi/2} 0 0" />
+        <origin xyz="0 0.14 0" rpy="-${pi/2} 0 0" />
         <axis xyz="0 0 1"/>
     </joint>
@@ -65,5 +65,5 @@
         <parent link="base_link"/>
         <child link="right_wheel"/>
-        <origin xyz="0 -0.175 0" rpy="${pi/2} 0 0" />
+        <origin xyz="0 -0.14 0" rpy="${pi/2} 0 0" />
         <axis xyz="0 0 -1"/>
     </joint>
